File: Precharger-v2-KiCAD/5V_Supply.sch (KiCad schematic (older format))
At the start: 6 parts

Commit message: Starting update with negative switching
Parts:
- U?: symbol General_Library:R-78HE5.0-0.3 -> Precharger-rescue:R-78HE5.0-0.3-General_Library
Changed lines of the file:
@@
 $EndComp
 $Comp
-L General_Library:R-78HE5.0-0.3 U?
+L Precharger-rescue:R-78HE5.0-0.3-General_Library U?
 U 1 1 5E058972
 P 6400 3900
