File: Precharger-v2-KiCAD/Voltage_Sensing.sch (KiCad schematic (older format))
At the start: 10 parts

Commit message: Starting update with negative switching
Connections:
- net +VSW renamed -VSW
Changed lines of the file:
@@
 Connection ~ 3900 4750
-$Comp
-L power:+VSW #PWR?
-U 1 1 5E0696C7
-P 2750 4050
-F 0 "#PWR?" H 2750 3900 50  0001 C CNN
-F 1 "+VSW" H 2765 4223 50  0000 C CNN
-F 2 "" H 2750 4050 50  0001 C CNN
-F 3 "" H 2750 4050 50  0001 C CNN
-	1    2750 4050
-	1    0    0    -1
-$EndComp
 $Comp
 L Connector:TestPoint TP?
@@
 	0    1    1    0
 $EndComp
+$Comp
+L power:-VSW #PWR?
+U 1 1 5E198C20
+P 2750 4050
+F 0 "#PWR?" H 2750 4150 50  0001 C CNN
+F 1 "-VSW" H 2765 4223 50  0000 C CNN
+F 2 "" H 2750 4050 50  0001 C CNN
+F 3 "" H 2750 4050 50  0001 C CNN
+	1    2750 4050
+	1    0    0    -1
+$EndComp
 $EndSCHEMATC
